File: Commodore-Vic-20.kicad_pcb (KiCad board)
At the start: 2 copper layers, 144 parts, among them CN1 Conn_01x03_Female, CN2 Conn_01x03_Male, P1 User Port, P10 Keyboard, P2 CONN_Cassette, P3 Serial, P4 Audio / Video, P5 Controller Port, P6 Expansion Port, P7 Power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

Commit message: replicate original board
Parts:
- removed CN2: Conn_01x03_Male, Connector_PinSocket_2.54mm:PinSocket_1x03_P2.54mm_Vertical
- removed D1: LED, LED_THT:LED_D5.0mm
- removed UC13: 74LS08, Package_DIP:DIP-14_W7.62mm
- removed UD4: 74LS04, Package_DIP:DIP-14_W7.62mm
- C15, C4, C42: footprint Capacitor_THT:CP_Radial_D5.0mm_P2.50mm -> Commodore:CP_Radial_D5.0mm_P5.0mm
- FB4, FB5, FB7, FB9: footprint Inductor_THT:L_Axial_L7.0mm_D3.3mm_P12.70mm_Horizontal_Fastron_MICC -> Inductor_THT:L_Axial_L7.0mm_D3.3mm_P5.08mm_Vertical_Fastron_MICC
- P1: footprint Connector_PinHeader_2.54mm:PinHeader_2x12_P2.54mm_Vertical -> Commodore:VC20_USERPORT
- P2: footprint Connector_PinHeader_2.54mm:PinHeader_2x06_P2.54mm_Vertical -> Commodore:VC20_CASSETTE
- P3: value Serial -> SERIAL; footprint Connector_PinHeader_2.54mm:PinHeader_1x06_P2.54mm_Vertical -> Commodore:DIN-6
- P4: footprint Connector_PinSocket_2.54mm:PinSocket_1x05_P2.54mm_Vertical -> Commodore:DIN-5
- P6: footprint Connector_PinHeader_2.54mm:PinHeader_2x21_P2.54mm_Vertical -> Commodore:VC20_EXPANSIONPORT
- P7: value Power -> POWER; footprint Connector_PinSocket_2.54mm:PinSocket_1x07_P2.54mm_Vertical -> Commodore:DIN-7
- Q1, Q3: footprint Package_TO_SOT_THT:TO-92_Inline -> Package_TO_SOT_THT:TO-92_Inline_Wide
- Q2: footprint Package_TO_SOT_THT:TO-220-3_Vertical -> Package_TO_SOT_THT:TO-92_Inline_Wide
- Q4: footprint Package_TO_SOT_THT:TO-92_Inline -> Package_TO_SOT_THT:TO-220-3_Vertical
- R11, R12, R13, R28, R7, R8, R9: footprint Resistor_THT:R_Axial_DIN0207_L6.3mm_D2.5mm_P10.16mm_Horizontal -> Resistor_THT:R_Axial_DIN0207_L6.3mm_D2.5mm_P5.08mm_Vertical
- UD7, UE11, UE12: footprint Package_DIP:DIP-24_W7.62mm -> Package_DIP:DIP-24_W15.24mm
- moved P7 563.0 mm to (395.5, 96.3), turned to 180 degrees
- moved R3 459.5 mm to (319.8, 136.3), turned to -90 degrees
- moved R2 456.7 mm to (316.9, 136.3), turned to -90 degrees
- moved R1 453.9 mm to (314.0, 136.3), turned to -90 degrees
- moved C36 439.4 mm to (370.3, 170.3)
- moved UE10 431.3 mm to (324.4, 143.9)
- moved P6 428.2 mm to (281.8, 116.5), turned to 90 degrees
- moved C1 423.0 mm to (324.3, 199.8)
- moved FB12 413.3 mm to (232.7, 201.5)
- moved U13 410.6 mm to (229.9, 133.5)
- moved C33 399.6 mm to (352.6, 171.8), turned to 180 degrees
- moved FB13 397.4 mm to (217.5, 201.5)
- moved CN1 396.4 mm to (362.9, 182.0), turned to -90 degrees
- moved UC3 385.3 mm to (235.3, 169.1)
- moved C27 384.9 mm to (302.5, 200.4)
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Connections:
- net Net-(F1-Pad1) renamed 9VACout
- net Net-(FB14-Pad1) renamed Serial_4
- net Net-(FB15-Pad1) renamed Serial_3
- net Net-(FB16-Pad1) renamed Serial_5
- net Net-(P4-Pin_3) renamed VIDEO_3
- net Net-(P7-9VAC-Pad6) renamed 9VACin
- net Net-(UAB1-CB1) renamed Serial_1
- net ~{RES} renamed Serial_6
- C12 pad 1: +5V -> GND
- C12 pad 2: GND -> +5V
- FB4 pad 1: Net-(FB4-Pad1) -> Net-(UB7-Ф1IN)
- FB4 pad 2: Net-(UB7-Ф1IN) -> Net-(FB4-Pad2)
- FB5 pad 1: Net-(FB5-Pad1) -> Net-(UB7-Ф2IN)
- FB5 pad 2: Net-(UB7-Ф2IN) -> Net-(FB5-Pad2)
- FB7 pad 1: Net-(C13-Pad2) -> Net-(UB7-COMP-C)
- FB7 pad 2: Net-(UB7-COMP-C) -> Net-(C13-Pad2)
- FB9 pad 1: Net-(Q1-C) -> Net-(UB7-VCC)
- FB9 pad 2: Net-(UB7-VCC) -> Net-(Q1-C)
- P10 pad 2: unconnected-(P10-Pad2) -> +5V
- P4 pad 4: Net-(P4-Pin_4) -> VIDEO_4
- P4 pad 5: Net-(P4-Pin_4) -> VIDEO_4
- P7 pad 4: Net-(P7-5V-Pad4) -> +5V
- P7 pad 5: Net-(P7-5V-Pad4) -> +5V
- Q2 pad 1: Net-(Q2-B) -> VIDEO_4
- Q2 pad 2: Net-(P4-Pin_4) -> Net-(Q1-C)
- Q2 pad 3: Net-(Q1-C) -> Net-(Q2-B)
- R11 pad 1: Net-(Q1-C) -> Net-(Q2-B)
- R11 pad 2: Net-(Q2-B) -> Net-(Q1-C)
- R12 pad 1: Net-(Q2-B) -> GND
- R12 pad 2: GND -> Net-(Q2-B)
- R13 pad 1: Net-(P4-Pin_4) -> GND
- R13 pad 2: GND -> VIDEO_4
- R28 pad 1: Net-(FB5-Pad1) -> Net-(FB5-Pad2)
- R7 pad 1: Net-(FB4-Pad1) -> Net-(FB4-Pad2)
- SW1 pad 3: Net-(P7-5V-Pad4) -> +5V
- U13 pad 10: (no net) -> Net-(UC4-O7)
- U13 pad 4: (no net) -> Net-(UC4-O4)
- U13 pad 5: (no net) -> Net-(UC4-O5)
- U13 pad 6: (no net) -> Net-(U15-~{CS})
- U13 pad 8: (no net) -> Net-(U14-~{CS})
- U13 pad 9: (no net) -> Net-(UC4-O6)
- UB4 pad 10: (no net) -> Net-(FB11-Pad2)
- UB4 pad 11: (no net) -> Net-(UD8-CE)
- UB9 pad 10: Net-(FB5-Pad1) -> Net-(FB5-Pad2)
- UB9 pad 13: Net-(FB4-Pad1) -> Net-(FB4-Pad2)
- UD7 pad 20: /VA12 -> /VA13
- UD7 pad 21: /VA13 -> /VA12
Routing:
- net IRQ: track 0.00 -> 286.2 mm, vias 0 -> 3
- net Serial_6: track 0.00 -> 261.8 mm, vias 0 -> 5
- net /CA4: track 0.00 -> 260.3 mm, vias 0 -> 3
- net /BD0: track 0.00 -> 259.4 mm, vias 0 -> 4
- net /BD1: track 0.00 -> 254.6 mm, vias 0 -> 4
- net NMI: track 0.00 -> 250.7 mm, vias 0 -> 2
- net /BD2: track 0.00 -> 249.8 mm, vias 0 -> 4
- net /CA2: track 0.00 -> 249.5 mm, vias 0 -> 2
- net /CA1: track 0.00 -> 248.2 mm, vias 0 -> 2
- net /CA3: track 0.00 -> 245.7 mm, vias 0 -> 1
- net /BD6: track 0.00 -> 243.8 mm, vias 0 -> 2
- net /BD5: track 0.00 -> 241.0 mm, vias 0 -> 2
- net /BD4: track 0.00 -> 234.9 mm, vias 0 -> 2
- net /BD3: track 0.00 -> 233.0 mm, vias 0 -> 2
- net /CA5: track 0.00 -> 201.3 mm, vias 0 -> 2
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Other:
- board outline added: 382.1 x 136.1 mm

Commit message: fix inductor
Parts:
- CR2: footprint Diode_THT:Diode_Bridge_15.1x15.1x6.3mm_P10.9mm -> Diode_THT:Diode_Bridge_Vishay_KBPM
- L4: footprint Inductor_THT:L_Axial_L6.6mm_D2.7mm_P10.16mm_Horizontal_Vishay_IM-2 -> Diode_THT:Diode_Bridge_15.1x15.1x6.3mm_P10.9mm
- moved FB2 431.2 mm to (355.0, 228.0)
- moved FB1 419.3 mm to (362.7, 178.7), turned to 90 degrees
- moved C38 390.7 mm to (370.5, 179.5)
- moved R23 390.6 mm to (357.6, 176.9), turned to 90 degrees
- moved C32 390.4 mm to (370.5, 151.3), turned to -90 degrees
- moved C31 390.2 mm to (370.3, 143.8), turned to 90 degrees
- moved C34 370.9 mm to (350.9, 163.8), turned to 180 degrees
- moved C10 304.3 mm to (252.7, 255.3)
- moved C13 304.3 mm to (260.9, 222.9)
- moved C17 304.3 mm to (260.9, 231.0)
- moved C20 304.3 mm to (260.9, 239.1)
- moved C21 304.3 mm to (260.9, 243.1)
- moved C25 304.3 mm to (260.9, 259.3)
- moved C40 304.3 mm to (277.2, 222.9)
- moved C44 304.3 mm to (277.2, 235.0)
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Routing:
- net L-PEN: track 14.5 -> 43.1 mm, vias 2 -> 3
- net +5V: track 173.6 -> 182.3 mm
- net Net-(FB1-Pad2): track 0.00 -> 5.34 mm

Commit message: dimension inductor
Parts:
- moved L4 21.6 mm to (362.6, 125.2), turned to -90 degrees
Changed lines of the file:
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@@
   )
   (footprint "Diode_THT:Diode_Bridge_15.1x15.1x6.3mm_P10.9mm" (layer "F.Cu")
-    (at 350.4404 143.1256)
+    (at 362.599 125.2334 -90)
     (descr "Single phase bridge rectifier case 15.1x15.1mm, pitch 10.9mm, see https://diotec.com/tl_files/diotec/files/pdf/datasheets/pb1000.pdf")
     (tags "Diode Bridge PB10xxS")
@@
     (property "Sheetname" "")
     (attr through_hole)
-    (fp_text reference "L4" (at 5.2 14.3 180) (layer "F.SilkS")
+    (fp_text reference "L4" (at 5.2 14.3 90) (layer "F.SilkS")
         (effects (font (size 1 1) (thickness 0.15)))
     )
-    (fp_text value "1m5" (at 5.2 -3.2 180) (layer "F.Fab")
+    (fp_text value "1m5" (at 5.2 -3.2 90) (layer "F.Fab")
         (effects (font (size 1 1) (thickness 0.15)))
     )
-    (fp_text user "${REFERENCE}" (at 5.2 5.415 180) (layer "F.Fab")
+    (fp_text user "${REFERENCE}" (at 5.2 5.415 90) (layer "F.Fab")
         (effects (font (size 1 1) (thickness 0.15)))
     )
@@
     (fp_line (start 13 13) (end -2.1 13)
       (stroke (width 0.12) (type solid)) (layer "F.Fab"))
-    (pad "1" thru_hole rect (at 0 0 180) (size 2.4 2.4) (drill 1.2) (layers "*.Cu" "*.Mask")
+    (pad "1" thru_hole rect (at 0 0 90) (size 2.4 2.4) (drill 1.2) (layers "*.Cu" "*.Mask")
       (net 44 "Net-(L4-Pad1)") (pinfunction "1") (pintype "passive"))
-    (pad "2" thru_hole circle (at 0.1 10.9 180) (size 2.4 2.4) (drill 1.2) (layers "*.Cu" "*.Mask")
+    (pad "2" thru_hole circle (at 0.1 10.9 90) (size 2.4 2.4) (drill 1.2) (layers "*.Cu" "*.Mask")
       (net 196 "Net-(C36-Pad1)") (pinfunction "2") (pintype "passive"))
-    (pad "3" thru_hole circle (at 10.9 10.9 180) (size 2.4 2.4) (drill 1.2) (layers "*.Cu" "*.Mask")
+    (pad "3" thru_hole circle (at 10.9 10.9 90) (size 2.4 2.4) (drill 1.2) (layers "*.Cu" "*.Mask")
       (net 22 "Net-(F1-Pad2)") (pinfunction "3") (pintype "passive"))
-    (pad "4" thru_hole circle (at 10.9 0 180) (size 2.4 2.4) (drill 1.2) (layers "*.Cu" "*.Mask")
+    (pad "4" thru_hole circle (at 10.9 0 90) (size 2.4 2.4) (drill 1.2) (layers "*.Cu" "*.Mask")
       (net 197 "Net-(C36-Pad2)") (pinfunction "4") (pintype "passive"))
     (model "${KICAD6_3DMODEL_DIR}/Diode_THT.3dshapes/Diode_Bridge_15.1x15.1x6.3mm_P10.9mm.wrl"
@@
       (effects (font (size 1 1) (thickness 0.15)))
     )
+    (format (prefix "") (suffix "") (units 3) (units_format 1) (precision 4))
+    (style (thickness 0.15) (arrow_length 1.27) (text_position_mode 0) (extension_height 0.58642) (extension_offset 0.5) keep_text_aligned)
+  )
+  (dimension (type aligned) (layer "User.4")
+    (pts (xy 349.6056 143.6624) (xy 349.6056 153.7716))
+    (height 3.2004)
+    (gr_text "10.1092 mm" (at 345.2552 148.717 90) (layer "User.4")
+      (effects (font (size 1 1) (thickness 0.15)))
+    )
+    (format (prefix "") (suffix "") (units 3) (units_format 1) (precision 4))
+    (style (thickness 0.15) (arrow_length 1.27) (text_position_mode 0) (extension_height 0.58642) (extension_offset 0.5) keep_text_aligned)
+  )
+  (dimension (type aligned) (layer "User.4")
+    (pts (xy 349.6056 143.6624) (xy 362.6612 143.6624))
+    (height -2.6924)
+    (gr_text "13.0556 mm" (at 356.1334 139.82) (layer "User.4")
+      (effects (font (size 1 1) (thickness 0.15)))
+    )

Commit message: develop rear of board
Parts:
- added JP1: power, Connector_PinSocket_2.54mm:PinSocket_1x02_P2.54mm_Vertical, F.Cu at (375.4, 172.0)
- added JP2: user, Connector_PinSocket_2.54mm:PinSocket_1x02_P2.54mm_Vertical, F.Cu at (39.9, 88.6)
- L4: footprint Diode_THT:Diode_Bridge_15.1x15.1x6.3mm_P10.9mm -> Diode_THT:Diode_Bridge_15.2x15.2x6.3mm_P10.9mm
- R27, R40, R5, R6: footprint Resistor_THT:R_Axial_DIN0207_L6.3mm_D2.5mm_P10.16mm_Horizontal -> Resistor_THT:R_Axial_DIN0207_L6.3mm_D2.5mm_P5.08mm_Vertical
- moved R6 187.1 mm to (202.2, 104.9), turned to 180 degrees
- moved R5 182.4 mm to (202.2, 108.2), turned to 180 degrees
- moved C10 174.9 mm to (143.5, 118.7), turned to 180 degrees
- moved C9 167.9 mm to (143.5, 123.7), turned to 180 degrees
- moved R40 141.5 mm to (138.7, 103.4)
- moved R27 113.6 mm to (138.4, 113.5)
- moved C25 38.4 mm to (260.9, 221.0)
- moved C3 32.8 mm to (261.2, 233.2)
- moved L3 28.8 mm to (357.4, 214.9)
- moved C6 24.0 mm to (241.8, 217.7)
- moved C5 24.0 mm to (241.8, 213.6)
- moved C7 24.0 mm to (241.8, 221.7)
- moved C8 24.0 mm to (241.8, 225.8)
- moved C50 22.9 mm to (270.3, 233.4)
- moved FB2 21.7 mm to (338.1, 214.4)
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Connections:
- F1 pad 1: 9VACout -> Net-(F1-Pad1)
- F1 pad 2: Net-(F1-Pad2) -> 9VACout
- L4 pad 3: Net-(F1-Pad2) -> Net-(F1-Pad1)
- R27 pad 1: Net-(Q1-E) -> GND
- R27 pad 2: GND -> Net-(Q1-E)
- R6 pad 1: Net-(C48-Pad2) -> Net-(R5-Pad2)
- R6 pad 2: Net-(R5-Pad1) -> Net-(C48-Pad2)
- SW1 pad 1: 9VACin -> Net-(L4-Pad1)
- SW1 pad 2: Net-(L4-Pad1) -> 9VACin
- SW1 pad 3: +5V -> Net-(C31-Pad2)
- SW1 pad 4: Net-(C31-Pad2) -> +5V
- UB9 pad 11: Net-(R5-Pad1) -> Net-(R5-Pad2)
- UB9 pad 12: Net-(R5-Pad1) -> Net-(R5-Pad2)
- UB9 pad 2: Net-(R5-Pad1) -> Net-(R5-Pad2)
- UB9 pad 3: Net-(R5-Pad1) -> Net-(R5-Pad2)
- UB9 pad 4: Net-(R5-Pad1) -> Net-(R5-Pad2)
- UB9 pad 5: Net-(R5-Pad2) -> Net-(R5-Pad1)
- UB9 pad 6: Net-(R5-Pad2) -> Net-(R5-Pad1)
- Y1 pad 1: Net-(R5-Pad2) -> Net-(R5-Pad1)
Routing:
- net GND: track 91.6 -> 1355.9 mm, vias 9 -> 17
- net +5V: track 182.3 -> 720.0 mm, vias 10 -> 17
- net JOY3: track 7.32 -> 446.5 mm, vias 0 -> 2
- net /CA4: track 260.3 -> 656.0 mm, vias 3 -> 7
- net /CA0: track 175.6 -> 526.2 mm, vias 2 -> 4
- net /CA1: track 248.2 -> 593.8 mm, vias 2 -> 4
- net /CA2: track 249.5 -> 584.6 mm, vias 2 -> 4
- net /CA3: track 245.7 -> 574.4 mm, vias 1 -> 3
- net SO2: track 72.1 -> 322.1 mm, vias 4 -> 6
- net Net-(U15-~{CS}): track 4.12 -> 227.5 mm, vias 1 -> 3
- net JOY2: track 6.86 -> 170.0 mm, vias 1 -> 4
- net JOY0: track 12.0 -> 173.3 mm, vias 1 -> 4
- net JOY1: track 9.40 -> 168.7 mm, vias 1 -> 4
- net L-PEN: track 43.1 -> 171.3 mm, vias 3 -> 5
- net Net-(P1-CB1): track 0.00 -> 102.4 mm, vias 0 -> 2
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- added copper zone on F.Cu, net GND
