File: Commodore-Vic-20.kicad_pcb (KiCad board)
At the start: 2 copper layers, 382.1 x 136.1 mm, 142 parts, among them CN1 Conn_01x03_Female, P1 User Port, P10 Keyboard, P2 CONN_Cassette, P3 SERIAL, P4 Audio / Video, P5 Controller Port, P6 Expansion Port, P7 POWER, Q1 2SC1815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

Commit message: more wiring
Parts:
- C11: footprint Capacitor_THT:CP_Radial_D5.0mm_P2.50mm -> Commodore:CP_Radial_D5.0mm_P5.0mm
- C50: footprint Capacitor_THT:C_Disc_D4.7mm_W2.5mm_P5.00mm -> Capacitor_THT:C_Disc_D4.3mm_W1.9mm_P5.00mm
- C6: footprint Capacitor_THT:C_Disc_D4.7mm_W2.5mm_P5.00mm -> Capacitor_THT:CP_Radial_D5.0mm_P2.50mm
- L3: footprint Inductor_THT:L_Axial_L6.6mm_D2.7mm_P10.16mm_Horizontal_Vishay_IM-2 -> Inductor_THT:L_Axial_L9.5mm_D4.0mm_P15.24mm_Horizontal_Fastron_SMCC
- moved C44 192.5 mm to (135.7, 88.4)
- moved C20 159.0 mm to (385.8, 144.0), turned to 90 degrees
- moved C21 156.8 mm to (380.5, 144.0), turned to 90 degrees
- moved C50 154.9 mm to (184.2, 104.7), turned to -90 degrees
- moved C25 130.3 mm to (136.4, 182.6), turned to 180 degrees
- moved C6 130.1 mm to (178.4, 104.1)
- moved C13 123.0 mm to (179.4, 113.5)
- moved C5 123.0 mm to (192.8, 100.8)
- moved C28 106.4 mm to (157.7, 187.7), turned to 180 degrees
- moved L3 78.1 mm to (375.4, 138.9), turned to -90 degrees
- moved R15 58.5 mm to (172.2, 201.2)
- moved R29 35.5 mm to (113.8, 202.4)
- moved L4 18.7 mm to (361.6, 143.9)
- moved R10 15.2 mm to (173.0, 114.3), turned to 90 degrees
- moved C48 13.9 mm to (187.0, 104.6)
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Connections:
- UE8 pad 11: VRW -> unconnected-(UE8-B7-Pad11)
Routing:
- net GND: track 1355.9 -> 2022.2 mm, vias 17 -> 22
- net +5V: track 720.0 -> 1205.0 mm, vias 17 -> 23
- net JOY0: track 173.3 -> 491.9 mm
- net JOY1: track 168.7 -> 486.5 mm
- net JOY2: track 170.0 -> 487.7 mm
- net L-PEN: track 171.3 -> 479.8 mm, vias 5 -> 6
- net /CA13: track 43.1 -> 309.6 mm, vias 1 -> 3
- net BLK4: track 184.9 -> 437.8 mm, vias 4 -> 6
- net Net-(UAB1-~{CS2}): track 36.8 -> 280.0 mm, vias 2 -> 4
- net CRW: track 159.4 -> 393.0 mm, vias 3 -> 5
- net VRW: track 132.2 -> 359.5 mm, vias 3 -> 6
- net Net-(P6-~{RES}): track 0.00 -> 196.9 mm, vias 0 -> 2
- net /BD7: track 160.0 -> 350.8 mm, vias 2 -> 3
- net Net-(UC4-O0): track 16.2 -> 201.3 mm, vias 0 -> 2
- net /CA12: track 169.7 -> 350.5 mm
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
Commit message: refresh project details
Parts:
- removed C17: 47u, Capacitor_THT:C_Disc_D4.7mm_W2.5mm_P5.00mm
- added C14: 47u, Commodore:CP_Radial_D5.0mm_P5.0mm, F.Cu at (161.9, 110.7)
- C4: footprint Commodore:CP_Radial_D5.0mm_P5.0mm -> Capacitor_THT:CP_Radial_D5.0mm_P2.50mm
- C7: footprint Capacitor_THT:C_Disc_D4.7mm_W2.5mm_P5.00mm -> Capacitor_THT:CP_Radial_D5.0mm_P2.50mm
- R41: footprint Resistor_THT:R_Axial_DIN0207_L6.3mm_D2.5mm_P10.16mm_Horizontal -> Resistor_THT:R_Axial_DIN0207_L6.3mm_D2.5mm_P5.08mm_Vertical
- moved R41 140.2 mm to (179.4, 123.5), turned to 90 degrees
- moved C7 126.6 mm to (184.1, 109.0), turned to 180 degrees
- moved C3 104.7 mm to (210.4, 141.6), turned to 90 degrees
- moved C8 99.2 mm to (195.2, 138.2)
- moved C40 89.3 mm to (352.4, 179.5), turned to 180 degrees
- moved FB2 36.8 mm to (363.3, 187.6), turned to 180 degrees
- moved C4 10.2 mm to (165.5, 101.2), turned to -90 degrees
- moved R10 7.68 mm to (180.1, 111.5), turned to 135 degrees
- moved C6 5.92 mm to (184.1, 105.6), turned to 180 degrees
- moved C12 5.58 mm to (161.2, 105.7), turned to 90 degrees
- moved C48 5.09 mm to (192.0, 105.9), turned to -75 degrees
- moved C50 3.89 mm to (187.8, 106.1)
- moved R6 3.20 mm to (202.3, 108.1)
- moved R5 3.18 mm to (202.3, 105.0)
Connections:
- R11 pad 1: Net-(Q2-B) -> Net-(Q1-C)
- R11 pad 2: Net-(Q1-C) -> Net-(Q2-B)
Routing:
- net L-PEN: track 479.8 -> 778.2 mm, vias 6 -> 10
- net Net-(CR2-+): track 130.5 -> 420.2 mm, vias 3 -> 7
- net Net-(P5-Pin_9): track 76.0 -> 315.4 mm, vias 1 -> 6
- net Net-(P5-Pin_5): track 78.5 -> 309.4 mm, vias 1 -> 6
- net GND: track 2022.2 -> 2244.5 mm, vias 22 -> 32
- net Net-(UE10-Ø0(IN)): track 150.1 -> 366.5 mm, vias 3 -> 9
- net +5V: track 1205.0 -> 1389.6 mm, vias 23 -> 28
- net BLK0: track 2.64 -> 168.7 mm, vias 1 -> 3
- net SO2: track 363.8 -> 484.7 mm, vias 6 -> 8
- net /CA0: track 526.2 -> 618.8 mm, vias 4 -> 6
- net VRW: track 359.5 -> 441.3 mm
- net Net-(UC4-O0): track 201.3 -> 269.3 mm
- net /CA4: track 792.8 -> 860.5 mm, vias 11 -> 13
- net CRW: track 393.0 -> 459.5 mm
- net /VA10: track 224.2 -> 287.4 mm
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
Commit message: add pdb render
Routing:
- net +5V: track 1389.6 -> 1449.7 mm, vias 28 -> 29
Changed lines of the file:
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@@
     )
   )
+  (gr_line (start 172.9994 105.9434) (end 172.9994 109.0422)
+    (stroke (width 0.15) (type default)) (layer "F.SilkS"))
   (gr_line (start 154.6352 83.5914) (end 154.6352 72.39)
     (stroke (width 0.1) (type default)) (layer "Edge.Cuts"))
@@
   (segment (start 271.4752 130.9516) (end 275.7274 130.9516) (width 0.2) (layer "F.Cu") (net 195))
   (segment (start 283.3724 128.5848) (end 283.4132 128.6256) (width 0.2) (layer "F.Cu") (net 195))
+  (segment (start 135.676 88.392) (end 128.778 88.392) (width 0.2) (layer "F.Cu") (net 195))
   (segment (start 34.036 151.638) (end 34.0868 151.6888) (width 0.2) (layer "F.Cu") (net 195))
   (segment (start 371.7944 156.2716) (end 373.126 154.94) (width 0.2) (layer "F.Cu") (net 195))
@@
   (segment (start 164.7952 156.5656) (end 179.324 156.5656) (width 0.2) (layer "F.Cu") (net 195))
   (segment (start 38.608 197.612) (end 50.038 197.612) (width 0.2) (layer "F.Cu") (net 195))
+  (segment (start 128.778 88.392) (end 128.7272 88.4428) (width 0.2) (layer "F.Cu") (net 195))
   (segment (start 78.0288 153.9748) (end 78.0288 152.0444) (width 0.5) (layer "F.Cu") (net 195))
   (via (at 311.5564 164.1348) (size 0.6) (drill 0.3) (layers "F.Cu" "B.Cu") (net 195))
   (via (at 255.4732 169.164) (size 0.6) (drill 0.3) (layers "F.Cu" "B.Cu") (net 195))
   (via (at 59.6392 152.0444) (size 0.6) (drill 0.3) (layers "F.Cu" "B.Cu") (net 195))
+  (via (at 128.7272 88.4428) (size 0.6) (drill 0.3) (layers "F.Cu" "B.Cu") (net 195))
   (via (at 135.0772 164.2364) (size 0.6) (drill 0.3) (layers "F.Cu" "B.Cu") (net 195))
   (via (at 50.292 201.676) (size 0.6) (drill 0.3) (layers "F.Cu" "B.Cu") (net 195))
@@
   (segment (start 93.98 103.5304) (end 91.3892 106.1212) (width 0.2) (layer "B.Cu") (net 195))
   (segment (start 93.3704 149.7076) (end 91.694 148.0312) (width 0.2) (layer "B.Cu") (net 195))
+  (segment (start 128.7272 88.4428) (end 128.7272 141.4272) (width 0.2) (layer "B.Cu") (net 195))
   (segment (start 193.548 156.718) (end 193.548 185.166) (width 0.2) (layer "B.Cu") (net 195))
   (segment (start 59.6392 149.1488) (end 59.6392 152.0444) (width 0.2) (layer "B.Cu") (net 195))
@@
   (segment (start 204.47 172.72) (end 204.47 182.626) (width 0.2) (layer "B.Cu") (net 195))
   (segment (start 112.268 156.7688) (end 109.4232 153.924) (width 0.2) (layer "B.Cu") (net 195))
+  (segment (start 128.7272 141.4272) (end 128.778 141.478) (width 0.2) (layer "B.Cu") (net 195))
   (segment (start 52.8828 153.924) (end 52.8828 151.6888) (width 0.2) (layer "B.Cu") (net 195))
   (segment (start 196.85 93.1926) (end 196.85 96.814) (width 0.2) (layer "B.Cu") (net 195))
