File: Commodore-Vic-20.kicad_pcb (KiCad board)
At the start: 2 copper layers, 382.1 x 136.1 mm, 142 parts, among them CN1 Conn_01x03_Female, P1 User Port, P10 Keyboard, P2 CONN_Cassette, P3 SERIAL, P4 Audio / Video, P5 Controller Port, P6 Expansion Port, P7 POWER, Q1 2SC1815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

Commit message: improve trace names
Connections:
- net Serial_6 renamed ~{RES}
