File: Commodore-Vic-20.kicad_sch (KiCad schematic)
At the start: 144 parts, among them CN1 Conn_01x03_Female, CN2 Conn_01x03_Male, P1 User Port, P10 Keyboard, P2 CONN_Cassette, P3 Serial, P4 Audio / Video, P5 Controller Port, P6 Expansion Port, P7 Power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

Commit message: replicate original board
Parts:
- removed CN2: Conn_01x03_Male, Connector_PinSocket_2.54mm:PinSocket_1x03_P2.54mm_Vertical, symbol Commodore-Vic-20-rescue:Conn_01x03_Male-Connector
- removed D1: LED, LED_THT:LED_D5.0mm, symbol Device:LED
- removed P3: Serial, Connector_PinHeader_2.54mm:PinHeader_1x06_P2.54mm_Vertical, symbol Commodore-Vic-20:CONN_Serial
- removed P4: Audio / Video, Connector_PinSocket_2.54mm:PinSocket_1x05_P2.54mm_Vertical, symbol Commodore-Vic-20-rescue:Conn_01x05_Female-Connector
- removed P7: Power, Connector_PinSocket_2.54mm:PinSocket_1x07_P2.54mm_Vertical, symbol Commodore-Vic-20:CONN_7_POWER
- removed Q2: 2SC1959, Package_TO_SOT_THT:TO-220-3_Vertical, symbol Transistor_BJT:2SC1945
- removed UD4: 74LS04, Package_DIP:DIP-14_W7.62mm, symbol 74xx:74LS04
- added P3: SERIAL, Commodore:DIN-6, symbol Connector:DIN-6
- added P4: Audio / Video, Commodore:DIN-5, symbol Connector:DIN-5_180degree
- added P7: POWER, Commodore:DIN-7, symbol Connector:DIN-7
- added Q2: 2SC1959, Package_TO_SOT_THT:TO-92_Inline_Wide, symbol Transistor_BJT:2SC1941
- added unit 5 of UB4
- C15, C4, C42: footprint Capacitor_THT:CP_Radial_D5.0mm_P2.50mm -> Commodore:CP_Radial_D5.0mm_P5.0mm
- FB4, FB5, FB7, FB9: footprint Inductor_THT:L_Axial_L7.0mm_D3.3mm_P12.70mm_Horizontal_Fastron_MICC -> Inductor_THT:L_Axial_L7.0mm_D3.3mm_P5.08mm_Vertical_Fastron_MICC
- P1: footprint Connector_PinHeader_2.54mm:PinHeader_2x12_P2.54mm_Vertical -> Commodore:VC20_USERPORT
- P2: footprint Connector_PinHeader_2.54mm:PinHeader_2x06_P2.54mm_Vertical -> Commodore:VC20_CASSETTE
- P6: footprint Connector_PinHeader_2.54mm:PinHeader_2x21_P2.54mm_Vertical -> Commodore:VC20_EXPANSIONPORT
- Q1, Q3: footprint Package_TO_SOT_THT:TO-92_Inline -> Package_TO_SOT_THT:TO-92_Inline_Wide
- Q4: footprint Package_TO_SOT_THT:TO-92_Inline -> Package_TO_SOT_THT:TO-220-3_Vertical
- R11, R12, R13, R28, R7, R8, R9: footprint Resistor_THT:R_Axial_DIN0207_L6.3mm_D2.5mm_P10.16mm_Horizontal -> Resistor_THT:R_Axial_DIN0207_L6.3mm_D2.5mm_P5.08mm_Vertical
- UD7, UE11, UE12: footprint Package_DIP:DIP-24_W7.62mm -> Package_DIP:DIP-24_W15.24mm
- renumbered UC13 to U13
Connections:
- net +5V: now also C12.2, P10.2, SW1.3, P4.1, P7.4, P7.5; no longer C12.1
- net GND: now also C12.1, R12.1, R13.1, P3.2, P4.2, P7.1, P7.2, P7.3; no longer C12.2, R12.2, R13.2
- net VA12: now also UD7.21 (CS2); no longer UD7.20 (CS1)
- net VA13: now also UD7.20 (CS1); no longer UD7.21 (CS2)
- net at UB7.2 (COMP-C): now also FB7.1; no longer FB7.2
- net at UB7.38 (Ф2IN): now also FB5.1; no longer FB5.2
- net at UB7.39 (Ф1IN): now also FB4.1; no longer FB4.2
- net at C8.1, FB6.2, UB7.40 (VCC): now also FB9.1; no longer FB9.2
- net at R7.1, UB9.13: now also FB4.2; no longer FB4.1
- net at R28.1, UB9.10: now also FB5.2; no longer FB5.1
- net at FB10.2, UC3.11, UD8.19 (CE)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: now also UB4.11
- net at FB11.2: now also UB4.10
- net at C15.1, C16.1, Q1.2 (C)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: now also FB9.2, R11.2, Q2.2 (C); no longer FB9.1, R11.1
- net VIDEO_3: now reaches C11.2
- net VIDEO_3: now also P4.3
- net at C13.2: now also FB7.2; no longer FB7.1
- net 9VACin: now reaches SW1.1
- net 9VACin: now also P7.6
- net 9VACout: now reaches F1.1
- net 9VACout: now also P7.7
- net Serial_1: now reaches UAB1.18 (CB1)
- net Serial_1: now also P3.1
- net Serial_3: now reaches FB15.1
- net Serial_3: now also P3.3
- net Serial_4: now reaches FB14.1
- net Serial_4: now also P3.4
- net Serial_5: now reaches FB16.1
- net Serial_5: now also P3.5
- net ~{RES} renamed Serial_6
- net Serial_6: now also P3.6
- new net: C17.1, Q2.3 (B), R11.1, R12.2
- new net VIDEO_4: P4.4, P4.5, Q2.1 (E), R13.2
- no-connect marks 11 -> 10
Other:
- moved on the sheet: C12, FB4, FB5, FB7, FB9

Commit message: fix inductor
Parts:
- CR2: footprint Diode_THT:Diode_Bridge_15.1x15.1x6.3mm_P10.9mm -> Diode_THT:Diode_Bridge_Vishay_KBPM
- L4: footprint Inductor_THT:L_Axial_L6.6mm_D2.7mm_P10.16mm_Horizontal_Vishay_IM-2 -> Diode_THT:Diode_Bridge_15.1x15.1x6.3mm_P10.9mm
Changed lines of the file:
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@@
       (effects (font (size 1.27 1.27)))
     )
-    (property "Footprint" "Inductor_THT:L_Axial_L6.6mm_D2.7mm_P10.16mm_Horizontal_Vishay_IM-2" (at 269.24 306.07 0)
+    (property "Footprint" "Diode_THT:Diode_Bridge_15.1x15.1x6.3mm_P10.9mm" (at 269.24 306.07 0)
       (effects (font (size 1.27 1.27)) hide)
     )
@@
       (effects (font (size 1.27 1.27)) (justify left))
     )
-    (property "Footprint" "Diode_THT:Diode_Bridge_15.1x15.1x6.3mm_P10.9mm" (at 298.45 306.07 0)
+    (property "Footprint" "Diode_THT:Diode_Bridge_Vishay_KBPM" (at 298.45 306.07 0)
       (effects (font (size 1.27 1.27)) hide)
     )

Commit message: dimension inductor
Parts:
- L4: footprint Diode_THT:Diode_Bridge_15.1x15.1x6.3mm_P10.9mm -> Diode_THT:Diode_Bridge_15.2x15.2x6.3mm_P10.9mm
Changed lines of the file:
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@@
       (effects (font (size 1.27 1.27)))
     )
-    (property "Footprint" "Diode_THT:Diode_Bridge_15.1x15.1x6.3mm_P10.9mm" (at 269.24 306.07 0)
+    (property "Footprint" "Diode_THT:Diode_Bridge_15.2x15.2x6.3mm_P10.9mm" (at 269.24 306.07 0)
       (effects (font (size 1.27 1.27)) hide)
     )

Commit message: develop rear of board
Parts:
- added JP1: power, Connector_PinSocket_2.54mm:PinSocket_1x02_P2.54mm_Vertical, symbol Connector:Conn_01x02_Socket
- added JP2: user, Connector_PinSocket_2.54mm:PinSocket_1x02_P2.54mm_Vertical, symbol Connector:Conn_01x02_Socket
- R27, R40, R5, R6: footprint Resistor_THT:R_Axial_DIN0207_L6.3mm_D2.5mm_P10.16mm_Horizontal -> Resistor_THT:R_Axial_DIN0207_L6.3mm_D2.5mm_P5.08mm_Vertical
Connections:
- net +5V: now also SW1.4; no longer SW1.3
- net 9VACin: now also SW1.2; no longer SW1.1
- net 9VACout: now also F1.2; no longer F1.1
- net GND: now also R27.1; no longer R27.2
- net at UB9.5, UB9.6, Y1.1: now also R5.1; no longer R5.2
- net at UB9.11, UB9.12, UB9.2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: now also R5.2, R6.1; no longer R5.1, R6.2
- net at C48.2, C50.2, UB9.1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: now also R6.2; no longer R6.1
- net at C11.1, Q1.1 (E): now also R27.2; no longer R27.1
- net at C31.2, L3.1: now also SW1.3; no longer SW1.4
- net at L4.3: now also F1.1; no longer F1.2
- net at L4.1: now also SW1.1; no longer SW1.2
- net at C36.1, CR2.3, L4.2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: now also JP2.1 (Pin_1)
- net at C36.2, CR2.4, L4.4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: now also JP2.2 (Pin_2)
Other:
- moved on the sheet: R5, R6
Changed lines of the file:
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@@
   (junction (at 425.45 144.78) (diameter 0) (color 0 0 0 0)
   )
+  (junction (at 171.45 438.15) (diameter 0) (color 0 0 0 0)
+  )
   (junction (at 668.02 114.3) (diameter 0) (color 0 0 0 0)
   )
@@
   (junction (at 105.41 40.64) (diameter 0) (color 0 0 0 0)
   )
+  (junction (at 173.99 440.69) (diameter 0) (color 0 0 0 0)
+  )
   (junction (at 190.5 313.69) (diameter 0) (color 0 0 0 0)
   )
@@
     (stroke (width 0) (type default))
   )
+  (wire (pts (xy 171.45 438.15) (xy 179.07 438.15))
+    (stroke (width 0) (type default))
+  )
   (wire (pts (xy 612.14 161.29) (xy 612.14 160.02))
     (stroke (width 0) (type default))
@@
     (stroke (width 0) (type default))
   )
-  (wire (pts (xy 171.45 438.15) (xy 179.07 438.15))
-    (stroke (width 0) (type default))
-  )
   (wire (pts (xy 272.415 73.025) (xy 270.51 73.025))
     (stroke (width 0) (type default))
@@
     (stroke (width 0) (type default))
   )
+  (wire (pts (xy 170.688 440.69) (xy 173.99 440.69))
+    (stroke (width 0) (type default))
+  )
   (wire (pts (xy 647.7 60.96) (xy 647.7 69.85))
     (stroke (width 0) (type default))
@@
     (stroke (width 0) (type default))
   )
+  (wire (pts (xy 170.688 438.15) (xy 171.45 438.15))
+    (stroke (width 0) (type default))
+  )
   (wire (pts (xy 624.84 175.26) (xy 629.92 175.26))
     (stroke (width 0) (type default))
@@
     )
   )
-  (symbol (lib_id "Device:R_US") (at 239.395 60.96 270) (unit 1)
+  (symbol (lib_id "Device:R_US") (at 239.395 60.96 90) (mirror x) (unit 1)
     (in_bom yes) (on_board yes) (dnp no)
     (property "Reference" "R5" (at 239.395 55.753 90)
@@
       (effects (font (size 1.27 1.27)))
     )
-    (property "Footprint" "Resistor_THT:R_Axial_DIN0207_L6.3mm_D2.5mm_P10.16mm_Horizontal" (at 239.141 61.976 90)
+    (property "Footprint" "Resistor_THT:R_Axial_DIN0207_L6.3mm_D2.5mm_P5.08mm_Vertical" (at 239.649 61.976 90)
       (effects (font (size 1.27 1.27)) hide)
     )
@@
     )
   )
-  (symbol (lib_id "Device:R_US") (at 265.43 61.595 270) (unit 1)
+  (symbol (lib_id "Device:R_US") (at 265.43 61.595 90) (mirror x) (unit 1)
     (in_bom yes) (on_board yes) (dnp no)
     (property "Reference" "R6" (at 265.43 56.388 90)
@@
       (effects (font (size 1.27 1.27)))
     )
-    (property "Footprint" "Resistor_THT:R_Axial_DIN0207_L6.3mm_D2.5mm_P10.16mm_Horizontal" (at 265.176 62.611 90)
+    (property "Footprint" "Resistor_THT:R_Axial_DIN0207_L6.3mm_D2.5mm_P5.08mm_Vertical" (at 265.684 62.611 90)
       (effects (font (size 1.27 1.27)) hide)
     )
@@
     )
   )
-  (symbol (lib_id "Device:R_US") (at 407.67 137.16 0) (unit 1)
+  (symbol (lib_id "Device:R_US") (at 407.67 137.16 0) (mirror x) (unit 1)
     (in_bom yes) (on_board yes) (dnp no)
-    (property "Reference" "R27" (at 405.9428 138.3284 0)
+    (property "Reference" "R27" (at 405.9428 135.9916 0)
       (effects (font (size 1.27 1.27)) (justify right))
     )
-    (property "Value" "470" (at 405.9428 136.017 0)
+    (property "Value" "470" (at 405.9428 138.303 0)
       (effects (font (size 1.27 1.27)) (justify right))
     )
-    (property "Footprint" "Resistor_THT:R_Axial_DIN0207_L6.3mm_D2.5mm_P10.16mm_Horizontal" (at 408.686 137.414 90)
+    (property "Footprint" "Resistor_THT:R_Axial_DIN0207_L6.3mm_D2.5mm_P5.08mm_Vertical" (at 408.686 136.906 90)
       (effects (font (size 1.27 1.27)) hide)
     )
@@
       (effects (font (size 1.27 1.27)) (justify right))
     )
-    (property "Footprint" "Resistor_THT:R_Axial_DIN0207_L6.3mm_D2.5mm_P10.16mm_Horizontal" (at 397.256 117.094 90)
+    (property "Footprint" "Resistor_THT:R_Axial_DIN0207_L6.3mm_D2.5mm_P5.08mm_Vertical" (at 397.256 117.094 90)
       (effects (font (size 1.27 1.27)) hide)
     )
@@
     )
   )
-  (symbol (lib_id "Device:Fuse_Small") (at 238.76 308.61 0) (unit 1)
+  (symbol (lib_id "Device:Fuse_Small") (at 238.76 308.61 0) (mirror y) (unit 1)
     (in_bom yes) (on_board yes) (dnp no)
     (property "Reference" "F1" (at 238.76 306.705 0)
@@
     )
   )
-  (symbol (lib_id "Switch:SW_DPST") (at 248.92 299.72 0) (unit 1)
+  (symbol (lib_id "Switch:SW_DPST") (at 248.92 299.72 0) (mirror y) (unit 1)
     (in_bom yes) (on_board yes) (dnp no)
     (property "Reference" "SW1" (at 248.92 293.8018 0)
@@
     )
   )
+  (symbol (lib_id "Connector:Conn_01x02_Socket") (at 344.424 310.134 0) (unit 1)
+    (in_bom yes) (on_board yes) (dnp no) (fields_autoplaced)
+    (property "Reference" "JP1" (at 345.186 310.769 0)
+      (effects (font (size 1.27 1.27)) (justify left))
+    )
+    (property "Value" "power" (at 345.186 313.309 0)
+      (effects (font (size 1.27 1.27)) (justify left))
+    )
+    (property "Footprint" "Connector_PinSocket_2.54mm:PinSocket_1x02_P2.54mm_Vertical" (at 344.424 310.134 0)
+      (effects (font (size 1.27 1.27)) hide)
+    )
+    (property "Datasheet" "~" (at 344.424 310.134 0)
+      (effects (font (size 1.27 1.27)) hide)
+    )
+    (pin "1")
+    (pin "2")
+    (instances
+      (project "Commodore-Vic-20"
+        (path "/12b7dc71-c774-4c36-b128-0efa0070fa41"
+          (reference "JP1") (unit 1)
+        )
+      )
+    )
+  )
   (symbol (lib_id "power:+5V") (at 143.51 294.64 90) (unit 1)
     (in_bom yes) (on_board yes) (dnp no)
@@
         )
       )
+    )
+  )
+  (symbol (lib_id "Connector:Conn_01x02_Socket") (at 165.608 438.15 0) (mirror y) (unit 1)
+    (in_bom yes) (on_board yes) (dnp no)
+    (property "Reference" "JP2" (at 164.846 438.785 0)
+      (effects (font (size 1.27 1.27)) (justify left))
+    )
+    (property "Value" "user" (at 164.846 441.325 0)
+      (effects (font (size 1.27 1.27)) (justify left))
+    )
+    (property "Footprint" "Connector_PinSocket_2.54mm:PinSocket_1x02_P2.54mm_Vertical" (at 165.608 438.15 0)
+      (effects (font (size 1.27 1.27)) hide)
+    )
+    (property "Datasheet" "~" (at 165.608 438.15 0)
+      (effects (font (size 1.27 1.27)) hide)
+    )
+    (pin "1")
+    (pin "2")
+    (instances
+      (project "Commodore-Vic-20"
+        (path "/12b7dc71-c774-4c36-b128-0efa0070fa41"
+          (reference "JP2") (unit 1)
+        )
+      )

Commit message: more wiring
Parts:
- C11: footprint Capacitor_THT:CP_Radial_D5.0mm_P2.50mm -> Commodore:CP_Radial_D5.0mm_P5.0mm
- C50: footprint Capacitor_THT:C_Disc_D4.7mm_W2.5mm_P5.00mm -> Capacitor_THT:C_Disc_D4.3mm_W1.9mm_P5.00mm
- C6: footprint Capacitor_THT:C_Disc_D4.7mm_W2.5mm_P5.00mm -> Capacitor_THT:CP_Radial_D5.0mm_P2.50mm
- L3: footprint Inductor_THT:L_Axial_L6.6mm_D2.7mm_P10.16mm_Horizontal_Vishay_IM-2 -> Inductor_THT:L_Axial_L9.5mm_D4.0mm_P15.24mm_Horizontal_Fastron_SMCC
Connections:
- net VRW: no longer UE8.11 (B7)
Changed lines of the file:
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@@
     (stroke (width 0) (type default))
   )
-  (bus_entry (at 167.64 189.23) (size 2.54 -2.54)
-    (stroke (width 0) (type default))
-  )
   (bus_entry (at 102.87 82.55) (size 2.54 -2.54)
     (stroke (width 0) (type default))
@@
     (stroke (width 0) (type default))
   )
-  (bus (pts (xy 170.18 181.61) (xy 170.18 186.69))
-    (stroke (width 0) (type default))
-  )
   (wire (pts (xy 330.2 128.27) (xy 307.34 128.27))
     (stroke (width 0) (type default))
@@
     (stroke (width 0) (type default))
   )
-  (wire (pts (xy 167.64 189.23) (xy 162.56 189.23))
-    (stroke (width 0) (type default))
-  )
   (bus (pts (xy 741.68 73.66) (xy 741.68 76.2))
     (stroke (width 0) (type default))
@@
     (effects (font (size 1.27 1.27)) (justify left bottom))
   )
-  (label "VRW" (at 162.56 189.23 0) (fields_autoplaced)
-    (effects (font (size 1.27 1.27)) (justify left bottom))
-  )
   (label "CA5" (at 744.22 86.36 0) (fields_autoplaced)
     (effects (font (size 1.27 1.27)) (justify left bottom))
@@
       (effects (font (size 1.27 1.27)) (justify left))
     )
-    (property "Footprint" "Capacitor_THT:C_Disc_D4.7mm_W2.5mm_P5.00mm" (at 358.14 94.2848 0)
+    (property "Footprint" "Capacitor_THT:CP_Radial_D5.0mm_P2.50mm" (at 358.14 94.2848 0)
       (effects (font (size 1.27 1.27)) hide)
     )
@@
       (effects (font (size 1.27 1.27)) (justify left))
     )
-    (property "Footprint" "Capacitor_THT:CP_Radial_D5.0mm_P2.50mm" (at 425.45 131.1148 0)
+    (property "Footprint" "Commodore:CP_Radial_D5.0mm_P5.0mm" (at 425.45 131.1148 0)
       (effects (font (size 1.27 1.27)) hide)
     )
@@
       (effects (font (size 1.27 1.27)))
     )
-    (property "Footprint" "Inductor_THT:L_Axial_L6.6mm_D2.7mm_P10.16mm_Horizontal_Vishay_IM-2" (at 266.7 297.18 0)
+    (property "Footprint" "Inductor_THT:L_Axial_L9.5mm_D4.0mm_P15.24mm_Horizontal_Fastron_SMCC" (at 266.7 297.18 0)
       (effects (font (size 1.27 1.27)) hide)
     )
@@
       (effects (font (size 1.27 1.27)))
     )
-    (property "Footprint" "Capacitor_THT:C_Disc_D4.7mm_W2.5mm_P5.00mm" (at 255.27 57.15 0)
+    (property "Footprint" "Capacitor_THT:C_Disc_D4.3mm_W1.9mm_P5.00mm" (at 255.27 57.15 0)
       (effects (font (size 1.27 1.27)) hide)
     )
