File: Commodore-Vic-20.kicad_sch (KiCad schematic)
At the start: 142 parts, among them CN1 Conn_01x03_Female, P1 User Port, P10 Keyboard, P2 CONN_Cassette, P3 SERIAL, P4 Audio / Video, P5 Controller Port, P6 Expansion Port, P7 POWER, Q1 2SC1815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

Commit message: resolve power circuit
Parts:
- added unit 2 of SW1
- CR2: symbol Device:D_Bridge_+-AA -> Device:D_Bridge_+AA-
- SW1: footprint Button_Switch_THT:SW_Push_2P1T_Toggle_CK_PVA1xxH1xxxxxxV2 -> Commodore:RockerSwitch_CuK_DPDT_E201J1AV2; symbol Switch:SW_DPST -> Switch:SW_DPDT_x2
Connections:
- net +5V: no longer P7.4, P7.5, SW1.4
- net 9VACin: now also SW1.4 (A); no longer SW1.2
- net GND: now also CR2.4 (-); no longer CR2.2 (-)
- net at C31.2, L3.1: now also SW1.2 (B); no longer SW1.3
- net at F1.1: now also L4.1; no longer L4.3
- net +5VP: now reaches SW1.1 (A)
- net +5VP: now also P7.4, P7.5; no longer L4.1
- net at C36.1, CR2.3, JP1.1 (Pin_1): now also L4.4; no longer L4.2
- net at C36.2, JP1.2 (Pin_2): now also CR2.2, L4.3; no longer CR2.4, L4.4
- new net: L4.2, SW1.5 (B)
- no-connect marks 10 -> 12
Other:
- moved on the sheet: C31, C32, L3
